Commit message: Two robots spawned and moving independently using teleop

File: install/swarm_robot_description/share/swarm_robot_description/urdf/turtlebot3_waffle_pi.urdf (robot description, URDF)
Before this commit: robot turtlebot3_waffle_pi, 11 links, 10 joints
Links:
- removed link ${namespace}base_footprint
- removed link ${namespace}base_link
- removed link ${namespace}base_scan
- removed link ${namespace}camera_link
- removed link ${namespace}camera_rgb_frame
- removed link ${namespace}camera_rgb_optical_frame
- removed link ${namespace}caster_back_left_link
- removed link ${namespace}caster_back_right_link
- removed link ${namespace}imu_link
- removed link ${namespace}wheel_left_link
- removed link ${namespace}wheel_right_link
- added link base_footprint
- added link base_link, mass 1.3729096e+00; collision box size=0.266 0.266 0.094; visual mesh filename=package://swarm_robot_description/meshes/bases/waffle_pi_ba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 scale=0.001 0.001 0.001
- added link base_scan, mass 0.114; collision cylinder length=0.0315 radius=0.055; visual mesh filename=package://swarm_robot_description/meshes/sensors/lds.stl scale=0.001 0.001 0.001
- added link camera_link; collision box size=0.015 0.030 0.027
- added link camera_rgb_frame
- added link camera_rgb_optical_frame
- added link caster_back_left_link, mass 0.005; collision box size=0.030 0.009 0.020
- added link caster_back_right_link, mass 0.005; collision box size=0.030 0.009 0.020
- added link imu_link
- added link wheel_left_link, mass 2.8498940e-02; collision cylinder length=0.018 radius=0.033; visual mesh filename=package://swarm_robot_description/meshes/wheels/left_tire.s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 scale=0.001 0.001 0.001
- added link wheel_right_link, mass 2.8498940e-02; collision cylinder length=0.018 radius=0.033; visual mesh filename=package://swarm_robot_description/meshes/wheels/right_tire.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 scale=0.001 0.001 0.001
Joints:
- removed joint ${namespace}base_joint
- removed joint ${namespace}camera_joint
- removed joint ${namespace}camera_rgb_joint
- removed joint ${namespace}camera_rgb_optical_joint
- removed joint ${namespace}caster_back_left_joint
- removed joint ${namespace}caster_back_right_joint
- removed joint ${namespace}imu_joint
- removed joint ${namespace}scan_joint
- removed joint ${namespace}wheel_left_joint
- removed joint ${namespace}wheel_right_joint
- added joint base_joint: type fixed, parent base_footprint, child base_link, origin xyz=0 0 0.010 rpy=0 0 0
- added joint camera_joint: type fixed, parent base_link, child camera_link, origin xyz=0.073 -0.011 0.084 rpy=0 0 0
- added joint camera_rgb_joint: type fixed, parent camera_link, child camera_rgb_frame, origin xyz=0.003 0.011 0.009 rpy=0 0 0
- added joint camera_rgb_optical_joint: type fixed, parent camera_rgb_frame, child camera_rgb_optical_frame, origin xyz=0 0 0 rpy=-1.57 0 -1.57
- added joint caster_back_left_joint: type fixed, parent base_link, child caster_back_left_link, origin xyz=-0.177 0.064 -0.004 rpy=-1.57 0 0
- added joint caster_back_right_joint: type fixed, parent base_link, child caster_back_right_link, origin xyz=-0.177 -0.064 -0.004 rpy=-1.57 0 0
- added joint imu_joint: type fixed, parent base_link, child imu_link, origin xyz=0.0 0 0.068 rpy=0 0 0
- added joint scan_joint: type fixed, parent base_link, child base_scan, origin xyz=-0.064 0 0.122 rpy=0 0 0
- added joint wheel_left_joint: type continuous, parent base_link, child wheel_left_link, origin xyz=0.0 0.144 0.023 rpy=-1.57 0 0, axis 0 0 1
- added joint wheel_right_joint: type continuous, parent base_link, child wheel_right_link, origin xyz=0.0 -0.144 0.023 rpy=-1.57 0 0, axis 0 0 1
